File: safety_board_Rev-A/safety_board_Rev-A.kicad_sch (KiCad schematic)
At the start: 21 parts, among them J1 24V_switched, J2 amp_A, J4 amp_B, J6 GND, J8 out_B, J9 out_A, K1 FINDER-40.52, Q1 2N7000

Commit message: Added images for the turn-on delay board, visual modifications to schematic.
Other:
- note added: "single throw dual pole switch -> connect to GND when switched off to discharge delay cap"
- note removed: "STDP switch -> connect to GND when switched off to discharge delay cap"
- moved on the sheet: C1, C2, C6, D1, D2, D4, H1, H2, J1, J2, J4, J6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
